File: TapClip32u4/tapclip.brd (EAGLE design)
At the start: 81 x 57.1 mm, 32 parts, among them X1 USBSMD, Y1 16MHz

Commit message: Keeping up with the Jones's
Parts:
- added C11, C12: (no value), SparkFun:0603-CAP
- added R4, R5, R6: (no value), SparkFun:0603-RES
- added U$13, U$14, U$15, U$16, U$17, U$18: ALLIGATOR_CLIP, sdgj:ALLIGATOR_CLIP
- added U$19, U$22: LTC1391-MUX, sdgj:SOIC16N
- added U$20: PGA112, sdgj:MICROSOIC10
- added U$21: ADG704-MUX, sdgj:MICROSOIC10
- U$2: value PGA116 -> ALLIGATOR_CLIP; device sdgj:TSSOP-20 -> sdgj:ALLIGATOR_CLIP
- moved U$2 55.1 mm to (3.81, -5.08), turned to 0 degrees
- moved U$10 49.0 mm to (73.7, 6.35)
- moved U$11 47.0 mm to (67.3, 6.35)
- moved U$9 44.5 mm to (7.62, 53.3)
- moved U$3 39.4 mm to (45.7, 53.3)
- moved U$8 30.5 mm to (14.0, 53.3)
- moved U$4 25.4 mm to (39.4, 53.3)
- moved U$12 22.9 mm to (52.1, 53.3)
- moved U$7 16.5 mm to (20.3, 53.3)
- moved RESET 13.0 mm to (25.4, 15.2), turned to 270 degrees
- moved U$5 11.4 mm to (33.0, 53.3)
- moved C2 8.89 mm to (34.3, 38.1), turned to 90 degrees
- moved ICSP 6.35 mm to (26.7, 27.9), turned to 90 degrees
- moved C10 5.73 mm to (40.8, 38.5)
- moved U$6 2.54 mm to (26.7, 53.3)
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Connections:
- removed net CS: U$2.P$18
- removed net EN: U$2.P$13
- removed net N$15: U$1.27
- new net CS1: U$19.11, U$22.11
- new net CS2: U$20.10
- new net D: R6.1, U$19.15, U$20.2, U$21.7, U$22.15
- new net MA0: U$1.27, U$21.1
- new net MA1: U$1.26, U$21.10
- new net MDOUT: U$19.13, U$22.12
- new net MS1: R4.2, U$21.2
- new net MS2: R4.1, R5.2, U$21.4
- new net MS3: R5.1, R6.2, U$21.9
- new net N$22: C2.1, U$19.16
- new net N$30: U$20.3
- new net N$36: U$21.5
- new net PB4: U$21.8
- new net S10: U$2.P$1, U$22.3
- new net S11: U$13.P$1, U$22.4
- new net S12: U$14.P$1, U$22.5
- new net S13: U$15.P$1, U$22.6
- new net S14: U$16.P$1, U$22.7
- new net S15: U$17.P$1, U$22.8
- new net S16: U$18.P$1
- new net SCLK: U$1.9, U$19.10, U$20.7, U$22.10
- net GND: now also C11.2, C12.2, U$19.14, U$19.9, U$20.4, U$20.6, U$21.3, U$22.14, U$22.9; no longer U$2.P$14
- net MISO: no longer U$2.P$17
- net MOSI: now also U$19.12, U$20.8; no longer U$2.P$16
- net N$14: now also C12.1, U$22.16; no longer U$1.26
- net S0: now also U$19.1; no longer U$2.P$7
- net S1: now also U$19.2; no longer U$2.P$6
- net S2: now also U$19.3; no longer U$2.P$5
- net S3: now also U$19.4; no longer U$2.P$4
- net S4: now also U$19.5; no longer U$2.P$3
- net S5: now also U$19.6; no longer U$2.P$2
- net S6: now also U$19.7; no longer U$2.P$20
- net S7: now also U$19.8; no longer U$2.P$10
- net S8: now also U$22.1; no longer U$2.P$11
- net S9: now also U$22.2; no longer U$2.P$12
- net SCK: no longer U$1.9, U$2.P$15
- net VCC: now also C11.1, U$20.1, U$20.9, U$21.6; no longer C2.1, U$2.P$1, U$2.P$19
- net VOUT: now also U$20.5; no longer U$2.P$8, U$2.P$9
Routing:
- net D: track 0.00 -> 27.9 mm
- net MISO: track 1.95 -> 22.8 mm
- net MOSI: track 0.00 -> 20.0 mm
- net VCC: track 33.1 -> 52.6 mm
- net SCLK: track 0.00 -> 18.1 mm, vias 0 -> 2
- net N$22: track 0.00 -> 2.77 mm
Other:
- board size 81 x 57.1 mm -> 78.4 x 57.1 mm

Commit message: Much has taken place here. Be still. Breath. Prepare yonder Gerbers.
Parts:
- removed RN1: 10K, resistor-dil:CAY16
- removed U$10, U$11, U$12, U$13, U$14, U$15, U$16, U$17, U$18, U$3, U$4, U$5, U$6, U$7, U$8, U$9: ALLIGATOR_CLIP, sdgj:ALLIGATOR_CLIP
- removed U$22: LTC1391-MUX, sdgj:SOIC16N
- added JP1: (no value), adafruit:1X06-CLEANBIG
- added LED3, LED4, LED5, LED6, LED7, LED8: GREEN, SparkFun:LED-0603
- added R20, R21, R22: 330, SparkFun-Passives:0402-RES
- added R8: (no value), SparkFun:0603-RES
- added S1, S2, S3, S4, S5, S6, S7, S8: ALLIGATOR_CLIP, sdgj:ALLIGATOR_CLIP
- added SJ1, SJ2: SOLDERJUMPERTRACE, SparkFun:SJ_2S-TRACE
- added SJ3, SJ4: SOLDERJUMPERNO, SparkFun:SJ_2S-NO
- C10, C11, C12, C2, C5: value (none) -> .1uF
- LED1: device SparkFun:LED-1206 -> SparkFun:LED-0603
- R3: value (none) -> 300
- U$2: value ALLIGATOR_CLIP -> LTC1391-MUX; device sdgj:ALLIGATOR_CLIP -> sdgj:SOIC16N
- moved C12 102.3 mm to (49.8, 25.3)
- moved U$2 53.8 mm to (44.5, 30.1), turned to 180 degrees
- moved C11 15.3 mm to (42.4, 20.1)
- moved C10 15.3 mm to (43.2, 23.4), turned to 0 degrees
- moved U$20 14.7 mm to (40.0, 22.5)
- moved C2 13.8 mm to (33.3, 24.4), turned to 0 degrees
- moved R6 12.1 mm to (55.9, 31.5), turned to 0 degrees
- moved C9 11.9 mm to (45.8, 20.1)
- moved C5 11.4 mm to (58.9, 8.64)
- moved ICSP 11.4 mm to (26.7, 16.5)
- moved U$1 11.4 mm to (50.8, 12.7)
- moved U$19 11.4 mm to (27.9, 29.2)
- moved C1 11.4 mm to (55.6, 20.6)
- moved C3 10.9 mm to (42.3, 13.0), turned to 180 degrees
- moved RESET 10.5 mm to (15.2, 12.7), turned to 180 degrees
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Connections:
- removed net N$14: C12.1, U$22.16
- removed net N$16: U$1.31
- removed net N$17: U$1.32
- removed net N$20: U$1.29
- removed net N$21: U$1.28
- removed net N$3: U$1.33
- removed net N$4: U$1.1
- removed net S10: U$2.P$1, U$22.3
- removed net S11: U$13.P$1, U$22.4
- removed net S12: U$14.P$1, U$22.5
- removed net S13: U$15.P$1, U$22.6
- removed net S14: U$16.P$1, U$22.7
- removed net S15: U$17.P$1, U$22.8
- removed net S16: U$18.P$1
- removed net S8: U$10.P$1, U$22.1
- removed net S9: U$11.P$1, U$22.2
- removed net SCK: ICSP.3
- new net J0: JP1.1, U$1.39
- new net J1: JP1.2, U$1.33
- new net J2: JP1.3, U$1.1
- new net J3: JP1.4, U$1.31
- new net J4: JP1.5, U$1.32
- new net J5: JP1.6, U$1.12
- new net LED0: R20.1, U$1.28
- new net LED1: R21.1, U$1.30
- new net LED2: R22.1, U$1.29
- new net N$15: S1.P$1, SJ2.2, SJ3.2
- new net N$24: LED5.A, LED6.C, LED7.A, LED8.C, R21.2
- new net N$25: LED3.A, LED4.C, LED7.C, LED8.A, R20.2
- new net N$26: LED3.C, LED4.A, LED5.C, LED6.A, R22.2
- new net VOUT1: U$1.40, U$2.15
- net CS1: now also U$2.11; no longer U$22.11
- net D: no longer U$22.15
- net GND: now also SJ4.1, U$2.14, U$2.9; no longer U$22.14, U$22.9
- net MA0: now also U$1.37; no longer U$1.27
- net MA1: now also U$1.38; no longer U$1.26
- net MDOUT: now also U$2.12; no longer U$22.12
- net N$18: now also U$1.36; no longer U$1.12
- net N$19: now also S2.P$1, SJ1.2, SJ4.2; no longer U$1.30
- net RESET: now also R8.1; no longer RN1.4
- net S0: now also S8.P$1, U$2.1; no longer U$12.P$1
- net S1: now also S7.P$1, U$2.2; no longer U$3.P$1
- net S2: now also S6.P$1, U$2.3; no longer U$4.P$1
- net S3: now also S5.P$1, U$2.4; no longer U$5.P$1
- net S4: now also S4.P$1, U$2.5; no longer U$6.P$1
- net S5: now also S3.P$1, U$2.6; no longer U$7.P$1
- net S6: now also SJ1.1, U$2.7; no longer U$8.P$1
- net S7: now also SJ2.1, U$2.8; no longer U$9.P$1
- net SCLK: now also ICSP.3, U$2.10; no longer U$22.10
- net VCC: now also C12.1, R8.2, SJ3.1, U$2.16; no longer RN1.5
Routing:
- net VCC: track 52.6 -> 135.6 mm, vias 0 -> 5
- net RESET: track 0.00 -> 55.5 mm, vias 0 -> 2
- net SCLK: track 18.1 -> 72.2 mm, vias 2 -> 0
- net J5: track 0.00 -> 49.3 mm, vias 0 -> 2
- net S0: track 0.00 -> 44.8 mm, vias 0 -> 2
- net S7: track 0.00 -> 38.4 mm, vias 0 -> 2
- net S5: track 0.00 -> 37.1 mm, vias 0 -> 1
- net J4: track 0.00 -> 34.1 mm, vias 0 -> 1
- net S4: track 0.00 -> 33.8 mm, vias 0 -> 1
- net S1: track 0.00 -> 33.2 mm, vias 0 -> 2
- net S6: track 0.00 -> 31.4 mm, vias 0 -> 2
- net S2: track 0.00 -> 29.7 mm, vias 0 -> 1
- net MOSI: track 20.0 -> 48.9 mm, vias 0 -> 2
- net J2: track 0.00 -> 28.9 mm, vias 0 -> 2
- net S3: track 0.00 -> 27.1 mm
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Other:
- board size 78.4 x 57.1 mm -> 70.2 x 46.3 mm
- board text added: "CUT FOR GND"
- board text added: "CUT FOR VCC"
- board text added: "GND"
- board text added: "StoryClip v.3"
- board text added: "VCC"
- board text added: "sjacoby@media.mit.edu"
- board text added: "| MIT Media Lab"

Commit message: And we've entered the rodeo.
Parts:
- added JP2: (no value), pinhead:1X02
- R8: value (none) -> 10k
- moved C11 2.13 mm to (42.5, 17.9)
- moved C9 0.43 mm to (45.6, 20.4)
- moved C12 0.22 mm to (49.7, 25.1)
Connections:
- removed net N$10: U$1.20
- removed net N$11: U$1.21
- removed net N$12: U$1.25
- removed net N$13: U$1.22
- removed net N$18: U$1.36
- removed net N$36: U$21.5
- removed net N$7: U$1.18
- removed net N$9: U$1.19
- removed net PB4: U$21.8
- new net ENMUX: U$1.39, U$21.5
- new net MUXIO: U$1.36, U$21.8
- net GND: now also JP2.2
- net J0: now also U$1.18; no longer U$1.39
- net J1: now also U$1.19; no longer U$1.33
- net J2: now also U$1.20; no longer U$1.1
- net J3: now also U$1.22; no longer U$1.31
- net J4: now also U$1.25; no longer U$1.32
- net J5: now also U$1.21; no longer U$1.12
- net LED1: now also U$1.31; no longer U$1.30
- net VCC: now also JP2.1
- net VOUT1: now also U$1.30; no longer U$1.40
Routing:
- net J1: track 15.1 -> 43.4 mm, vias 0 -> 1
- net J0: track 21.2 -> 44.2 mm, vias 2 -> 1
- net ENMUX: track 0.00 -> 17.0 mm, vias 0 -> 2
- net VOUT1: track 9.98 -> 25.7 mm, vias 0 -> 2
- net J5: track 49.3 -> 34.8 mm, vias 2 -> 1
- net MUXIO: track 0.00 -> 14.0 mm, vias 0 -> 2
- net J2: track 28.9 -> 41.1 mm, vias 2 -> 1
- net J3: track 23.5 -> 30.8 mm, vias 0 -> 1
- net VCC: track 135.6 -> 142.8 mm, vias 5 -> 2
- net CS2: track 0.00 -> 4.80 mm
- net J4: track 34.1 -> 30.0 mm
- net SCLK: track 72.2 -> 68.7 mm
- net D: track 35.4 -> 38.5 mm
- net S4: track 33.8 -> 31.2 mm
- net MOSI: track 48.9 -> 47.0 mm
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- added copper zone on layer 1, net GND
- added copper zone on layer 16, net GND
Other:
- board text added: "J0"

Commit message: These are the things that should be done for this.
Connections:
- net CS2: now also U$1.1
Routing:
- net CS2: track 4.80 -> 5.72 mm
